Commit message: fixed valkyrie URDF model for pinocchio

File: share/urdf/valkyrie_sim.urdf (robot description, URDF)
Before this commit: robot valkyrie, 80 links, 79 joints
Joints:
- joint hokuyo_joint: type continuous -> fixed
- joint leftIndexFingerPitch1: type revolute -> fixed
- joint leftIndexFingerPitch2: type revolute -> fixed
- joint leftIndexFingerPitch3: type revolute -> fixed
- joint leftMiddleFingerPitch1: type revolute -> fixed
- joint leftMiddleFingerPitch2: type revolute -> fixed
- joint leftMiddleFingerPitch3: type revolute -> fixed
- joint leftPinkyPitch1: type revolute -> fixed
- joint leftPinkyPitch2: type revolute -> fixed
- joint leftPinkyPitch3: type revolute -> fixed
- joint leftThumbPitch1: type revolute -> fixed
- joint leftThumbPitch2: type revolute -> fixed
- joint leftThumbPitch3: type revolute -> fixed
- joint leftThumbRoll: type revolute -> fixed
- joint rightIndexFingerPitch1: type revolute -> fixed
- joint rightIndexFingerPitch2: type revolute -> fixed
- joint rightIndexFingerPitch3: type revolute -> fixed
- joint rightMiddleFingerPitch1: type revolute -> fixed
- joint rightMiddleFingerPitch2: type revolute -> fixed
- joint rightMiddleFingerPitch3: type revolute -> fixed
- joint rightPinkyPitch1: type revolute -> fixed
- joint rightPinkyPitch2: type revolute -> fixed
- joint rightPinkyPitch3: type revolute -> fixed
- joint rightThumbPitch1: type revolute -> fixed
- joint rightThumbPitch2: type revolute -> fixed
- joint rightThumbPitch3: type revolute -> fixed
- joint rightThumbRoll: type revolute -> fixed

Commit message: fix for pinocchio wrapper with continuous joints by tavu

File: share/urdf/valkyrie_sim.urdf (robot description, URDF)
Before this commit: robot valkyrie, 80 links, 79 joints
Joints:
- joint hokuyo_joint: type fixed -> continuous
- joint leftIndexFingerPitch1: type fixed -> revolute
- joint leftIndexFingerPitch2: type fixed -> revolute
- joint leftIndexFingerPitch3: type fixed -> revolute
- joint leftMiddleFingerPitch1: type fixed -> revolute
- joint leftMiddleFingerPitch2: type fixed -> revolute
- joint leftMiddleFingerPitch3: type fixed -> revolute
- joint leftPinkyPitch1: type fixed -> revolute
- joint leftPinkyPitch2: type fixed -> revolute
- joint leftPinkyPitch3: type fixed -> revolute
- joint leftThumbPitch1: type fixed -> revolute
- joint leftThumbPitch2: type fixed -> revolute
- joint leftThumbPitch3: type fixed -> revolute
- joint leftThumbRoll: type fixed -> revolute
- joint rightIndexFingerPitch1: type fixed -> revolute
- joint rightIndexFingerPitch2: type fixed -> revolute
- joint rightIndexFingerPitch3: type fixed -> revolute
- joint rightMiddleFingerPitch1: type fixed -> revolute
- joint rightMiddleFingerPitch2: type fixed -> revolute
- joint rightMiddleFingerPitch3: type fixed -> revolute
- joint rightPinkyPitch1: type fixed -> revolute
- joint rightPinkyPitch2: type fixed -> revolute
- joint rightPinkyPitch3: type fixed -> revolute
- joint rightThumbPitch1: type fixed -> revolute
- joint rightThumbPitch2: type fixed -> revolute
- joint rightThumbPitch3: type fixed -> revolute
- joint rightThumbRoll: type fixed -> revolute
