Commit message: Added Contact EKF

File: share/urdf/nao.urdf (robot description, URDF)
Before this commit: robot NaoH25V40, 84 links, 83 joints
Links:
- removed link CameraBottom_frame
- removed link CameraBottom_optical_frame
- removed link CameraTop_frame
- removed link CameraTop_optical_frame
- removed link ChestButton_frame
- removed link HeadTouchFront_frame
- removed link HeadTouchMiddle_frame
- removed link HeadTouchRear_frame
- removed link ImuTorsoAccelerometer_frame
- removed link ImuTorsoGyrometer_frame
- removed link LFinger11_link
- removed link LFinger12_link
- removed link LFinger13_link
- removed link LFinger21_link
- removed link LFinger22_link
- removed link LFinger23_link
- removed link LFootBumperLeft_frame
- removed link LFootBumperRight_frame
- removed link LFsrFL_frame
- removed link LFsrFR_frame
- removed link LFsrRL_frame
- removed link LFsrRR_frame
- removed link LHandTouchBack_frame
- removed link LHandTouchLeft_frame
- removed link LHandTouchRight_frame
- removed link LInfraRed_frame
- removed link LSonar_frame
- removed link LThumb1_link
- removed link LThumb2_link
- removed link LaserHead_frame
- removed link MicroFrontCenter_frame
- removed link MicroRearCenter_frame
- removed link MicroSurroundLeft_frame
- removed link MicroSurroundRight_frame
- removed link RFinger11_link
- removed link RFinger12_link
- removed link RFinger13_link
- removed link RFinger21_link
- removed link RFinger22_link
- removed link RFinger23_link
- removed link RFootBumperLeft_frame
- removed link RFootBumperRight_frame
- removed link RFsrFL_frame
- removed link RFsrFR_frame
- removed link RFsrRL_frame
- removed link RFsrRR_frame
- removed link RHandTouchBack_frame
- removed link RHandTouchLeft_frame
- removed link RHandTouchRight_frame
- removed link RInfraRed_frame
- removed link RSonar_frame
- removed link RThumb1_link
- removed link RThumb2_link
Joints:
- removed joint Accelerometer_sensor_fixedjoint
- removed joint CameraBottom_optical_frame_fixedjoint
- removed joint CameraBottom_sensor_fixedjoint
- removed joint CameraTop_optical_frame_fixedjoint
- removed joint CameraTop_sensor_fixedjoint
- removed joint ChestBoard/Button_sensor_fixedjoint
- removed joint Gyrometer_sensor_fixedjoint
- removed joint Head/LaserHead
- removed joint Head/Touch/Front_sensor_fixedjoint
- removed joint Head/Touch/Middle_sensor_fixedjoint
- removed joint Head/Touch/Rear_sensor_fixedjoint
- removed joint InfraredL_sensor_fixedjoint
- removed joint InfraredR_sensor_fixedjoint
- removed joint LFinger11
- removed joint LFinger12
- removed joint LFinger13
- removed joint LFinger21
- removed joint LFinger22
- removed joint LFinger23
- removed joint LFoot/Bumper/Left_sensor_fixedjoint
- removed joint LFoot/Bumper/Right_sensor_fixedjoint
- removed joint LFoot/FSR/FrontLeft_sensor_fixedjoint
- removed joint LFoot/FSR/FrontRight_sensor_fixedjoint
- removed joint LFoot/FSR/RearLeft_sensor_fixedjoint
- removed joint LFoot/FSR/RearRight_sensor_fixedjoint
- removed joint LHand/Touch/Back_sensor_fixedjoint
- removed joint LHand/Touch/Left_sensor_fixedjoint
- removed joint LHand/Touch/Right_sensor_fixedjoint
- removed joint LThumb1
- removed joint LThumb2
- removed joint MicroFront_sensor_fixedjoint
- removed joint MicroLeft_sensor_fixedjoint
- removed joint MicroRear_sensor_fixedjoint
- removed joint MicroRight_sensor_fixedjoint
- removed joint RFinger11
- removed joint RFinger12
- removed joint RFinger13
- removed joint RFinger21
- removed joint RFinger22
- removed joint RFinger23
- removed joint RFoot/Bumper/Left_sensor_fixedjoint
- removed joint RFoot/Bumper/Right_sensor_fixedjoint
- removed joint RFoot/FSR/FrontLeft_sensor_fixedjoint
- removed joint RFoot/FSR/FrontRight_sensor_fixedjoint
- removed joint RFoot/FSR/RearLeft_sensor_fixedjoint
- removed joint RFoot/FSR/RearRight_sensor_fixedjoint
- removed joint RHand/Touch/Back_sensor_fixedjoint
- removed joint RHand/Touch/Left_sensor_fixedjoint
- removed joint RHand/Touch/Right_sensor_fixedjoint
- removed joint RThumb1
- removed joint RThumb2
- removed joint Sonar/Left_sensor_fixedjoint
- removed joint Sonar/Right_sensor_fixedjoint
