Commit message: removed hokuyo frame (lidar)

File: urdf/valk.urdf (robot description, URDF)
Before this commit: robot valkyrie, 80 links, 79 joints
Links:
- removed link head_hokuyo_frame
- removed link hokuyo_link
Joints:
- removed joint head_hokuyo_joint
- removed joint hokuyo_joint

Commit message: removed links and joints of fingers for compatibility with fast joint state topic

File: urdf/valk.urdf (robot description, URDF)
Before this commit: robot valkyrie, 78 links, 77 joints
Links:
- removed link leftIndexFingerPitch1Link
- removed link leftIndexFingerPitch2Link
- removed link leftIndexFingerPitch3Link
- removed link leftMiddleFingerPitch1Link
- removed link leftMiddleFingerPitch2Link
- removed link leftMiddleFingerPitch3Link
- removed link leftPinkyPitch1Link
- removed link leftPinkyPitch2Link
- removed link leftPinkyPitch3Link
- removed link leftThumbPitch1Link
- removed link leftThumbPitch2Link
- removed link leftThumbPitch3Link
- removed link leftThumbRollLink
- removed link rightIndexFingerPitch1Link
- removed link rightIndexFingerPitch2Link
- removed link rightIndexFingerPitch3Link
- removed link rightMiddleFingerPitch1Link
- removed link rightMiddleFingerPitch2Link
- removed link rightMiddleFingerPitch3Link
- removed link rightPinkyPitch1Link
- removed link rightPinkyPitch2Link
- removed link rightPinkyPitch3Link
- removed link rightThumbPitch1Link
- removed link rightThumbPitch2Link
- removed link rightThumbPitch3Link
- removed link rightThumbRollLink
Joints:
- removed joint leftIndexFingerPitch1
- removed joint leftIndexFingerPitch2
- removed joint leftIndexFingerPitch3
- removed joint leftMiddleFingerPitch1
- removed joint leftMiddleFingerPitch2
- removed joint leftMiddleFingerPitch3
- removed joint leftPinkyPitch1
- removed joint leftPinkyPitch2
- removed joint leftPinkyPitch3
- removed joint leftThumbPitch1
- removed joint leftThumbPitch2
- removed joint leftThumbPitch3
- removed joint leftThumbRoll
- removed joint rightIndexFingerPitch1
- removed joint rightIndexFingerPitch2
- removed joint rightIndexFingerPitch3
- removed joint rightMiddleFingerPitch1
- removed joint rightMiddleFingerPitch2
- removed joint rightMiddleFingerPitch3
- removed joint rightPinkyPitch1
- removed joint rightPinkyPitch2
- removed joint rightPinkyPitch3
- removed joint rightThumbPitch1
- removed joint rightThumbPitch2
- removed joint rightThumbPitch3
- removed joint rightThumbRoll
