Commit message: added sole below the ankle roll

File: urdf/g1_12dof.urdf (robot description, URDF)
Before this commit: robot g1_12dof, 31 links, 30 joints
Links:
- added link left_foot_sole
- added link right_foot_sole
Joints:
- added joint left_foot_sole_joint: type fixed, parent left_ankle_roll_link, child left_foot_sole, origin xyz=0.1 0 -0.035 rpy=0 0 0
- added joint right_foot_sole_joint: type fixed, parent right_ankle_roll_link, child right_foot_sole, origin xyz=0.10 0 -0.035 rpy=0 0 0
